File: fourkey.kicad_pcb (KiCad board)
At the start: 2 copper layers, 85.3 x 77.7 mm, 23 parts, among them K1 KEYSW, K2 KEYSW, K3 KEYSW, K4 KEYSW, SW1 SW_PUSH, U1 ProMicro

Commit message: add some labels
Parts:
- SW1: value SW_PUSH -> RESET
Other:
- board text added: "CAMERA"
- board text added: "HAND"
- board text added: "MIC"
- board text added: "RAW"
- board text added: "TXO"
- board text added: "VIEW"
Changed lines of the file:
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@@
   (general
     (thickness 1.6)
-    (drawings 69)
+    (drawings 75)
     (tracks 46)
     (zones 0)
@@
     (34 B.Paste user)
     (35 F.Paste user)
-    (36 B.SilkS user hide)
+    (36 B.SilkS user)
     (37 F.SilkS user)
     (38 B.Mask user)
@@
       (effects (font (size 1 1) (thickness 0.15)))
     )
-    (fp_text value SW_PUSH (at 0 3.75) (layer F.SilkS)
+    (fp_text value RESET (at 0 3.75 180) (layer F.SilkS)
       (effects (font (size 1 1) (thickness 0.15)))
     )
@@
     )
   )
+  (gr_text TXO (at 72.39 73.914 180) (layer F.SilkS)
+    (effects (font (size 1 0.7) (thickness 0.15)))
+  )
+  (gr_text RAW (at 72.39 85.09) (layer F.SilkS)
+    (effects (font (size 1 0.7) (thickness 0.15)))
+  )
+  (gr_text MIC (at 134.643 115.062) (layer B.SilkS)
+    (effects (font (size 2 1.5) (thickness 0.15)) (justify mirror))
+  )
+  (gr_text HAND (at 115.593 115.062) (layer B.SilkS)
+    (effects (font (size 2 1.5) (thickness 0.15)) (justify mirror))
+  )
+  (gr_text CAMERA (at 96.543 115.062) (layer B.SilkS)
+    (effects (font (size 2 1.5) (thickness 0.15)) (justify mirror))
+  )
+  (gr_text VIEW (at 77.492999 115.062) (layer B.SilkS)
+    (effects (font (size 2 1.5) (thickness 0.15)) (justify mirror))
+  )
   (gr_line (start 127.643 98.298) (end 127.643 111.297999) (layer Edge.Cuts) (width 0.2))
   (gr_line (start 141.643 111.297999) (end 141.643 98.298) (layer Edge.Cuts) (width 0.2))
@@
   (gr_arc (start 90.043 98.298) (end 90.043 97.798) (angle -90) (layer Edge.Cuts) (width 0.2))
   (gr_line (start 128.143 111.797999) (end 141.143 111.797999) (layer Edge.Cuts) (width 0.2))
-  (gr_text github.com/trepmal/fourkey (at 94.996 54.356) (layer B.SilkS)
-    (effects (font (size 1 1) (thickness 0.15)) (justify mirror))
+  (gr_text github.com/trepmal/fourkey (at 88.9 54.356) (layer B.SilkS)
+    (effects (font (size 2 1.5) (thickness 0.15)) (justify mirror))
   )
   (gr_arc (start 147.844 66.834) (end 148.844 66.834) (angle 90) (layer Edge.Cuts) (width 0.05))
